Commit message: Error Debug

File: urdf/husky.urdf (robot description, URDF)
Before this commit: robot husky_reduced, 18 links, 17 joints
Links:
- link bl_ankle1: geometry collision mesh filename=package://husky/meshes/bl_ankle1.STL; visual mesh filename=package://husky/meshes/bl_ankle1.STL
- link bl_femur: geometry collision mesh filename=package://husky/meshes/bl_femur.STL; visual mesh filename=package://husky/meshes/bl_femur.STL
- link bl_hip: geometry collision mesh filename=package://husky/meshes/bl_hip.STL; visual mesh filename=package://husky/meshes/bl_hip.STL
- link bl_tibia: geometry collision mesh filename=package://husky/meshes/bl_tibia.STL; visual mesh filename=package://husky/meshes/bl_tibia.STL
- link body_link: geometry collision mesh filename=package://husky/meshes/body_link.STL; visual mesh filename=package://husky/meshes/body_link.STL
- link br_ankle: geometry collision mesh filename=package://husky/meshes/br_ankle.STL; visual mesh filename=package://husky/meshes/br_ankle.STL
- link br_femur: geometry collision mesh filename=package://husky/meshes/br_femur.STL; visual mesh filename=package://husky/meshes/br_femur.STL
- link br_hip: geometry collision mesh filename=package://husky/meshes/br_hip.STL; visual mesh filename=package://husky/meshes/br_hip.STL
- link br_tibia: geometry collision mesh filename=package://husky/meshes/br_tibia.STL; visual mesh filename=package://husky/meshes/br_tibia.STL
- link fl_ankle1: geometry collision mesh filename=package://husky/meshes/fl_ankle1.STL; visual mesh filename=package://husky/meshes/fl_ankle1.STL
- link fl_femur: geometry collision mesh filename=package://husky/meshes/fl_femur.STL; visual mesh filename=package://husky/meshes/fl_femur.STL
- link fl_hip: geometry collision mesh filename=package://husky/meshes/fl_hip.STL; visual mesh filename=package://husky/meshes/fl_hip.STL
- link fl_tibia: geometry collision mesh filename=package://husky/meshes/fl_tibia.STL; visual mesh filename=package://husky/meshes/fl_tibia.STL
- link fr_ankle1: geometry collision mesh filename=package://husky/meshes/fr_ankle1.STL; visual mesh filename=package://husky/meshes/fr_ankle1.STL
- link fr_femur: geometry collision mesh filename=package://husky/meshes/fr_femur.STL; visual mesh filename=package://husky/meshes/fr_femur.STL
- link fr_hip: geometry collision mesh filename=package://husky/meshes/fr_hip.STL; visual mesh filename=package://husky/meshes/fr_hip.STL
- link fr_tibia: geometry collision mesh filename=package://husky/meshes/fr_tibia.STL; visual mesh filename=package://husky/meshes/fr_tibia.STL
Joints:
- removed joint br_ankle
- added joint br_ankle1: type revolute, parent br_tibia, child br_ankle, origin xyz=0.332999999999973 0 0 rpy=-3.12284991813426 -0.0144859149234315 1.29924335391435, axis 0 0 1, limit lower=-3.1416 upper=3.1416 effort=1000 velocity=1000
